Commit message: added imu link visuals

File: src/roverrobotics_description/urdf/accessories/imu.urdf (robot description, URDF)
Before this commit: robot imu, 1 links, 1 joints
Links:
- link imu_link: geometry visual mesh filename=file://$(find roverrobotics_description)/meshes/BNO055.stl scale=0.001 0.001 0.001
Joints:
- joint imu_to_payload: origin xyz=0 0 0 rpy=0 0 0 -> xyz=-0.190 0 0.081 rpy=0 0 0
