Commit message: Refactor code structure for improved readability and maintainability changed back to real hardware

File: src/roverrobotics_description/urdf/accessories/realsense_camera.urdf (robot description, URDF)
Before this commit: robot imu, 2 links, 2 joints
Links:
- removed link realsense_camera_link
- removed link realsense_camera_link_optical
- added link camera_link, mass 0.072; collision box size=0.025 0.09 0.025; visual mesh filename=file://$(find roverrobotics_description)/meshes/d435.dae scale=1.0 1.0 1.0
Joints:
- removed joint realsense_camera_joint
- removed joint realsense_camera_optical_joint
- added joint camera_joint: type fixed, parent payload_link, child camera_link, origin xyz=0.215 0 0.065 rpy=0 0 0
