Commit message: experiment development

File: src/roverrobotics_description/urdf/rover_2wd.urdf (robot description, URDF)
Before this commit: robot rover_2wd, 8 links, 7 joints
Links:
- added link base_footprint
Joints:
- added joint base_footprint_to_base_link: type fixed, parent base_footprint, child base_link, origin xyz=0 0 0 rpy=0 0 0, axis 0 0 1

Commit message: Added gitignoe fixed base_footprint and base_link relations

File: src/roverrobotics_description/urdf/rover_2wd.urdf (robot description, URDF)
Before this commit: robot rover_2wd, 9 links, 8 joints
Joints:
- joint base_footprint_to_base_link: child base_link -> base_footprint; parent base_footprint -> base_link
